File: support_docs/board_layouts/cape 0.0/t1.brd (EAGLE design)
At the start: 100 x 80 mm, 14 parts, among them IC1 74HC595N

Commit message: testing and updating cape layout
Parts:
- added LED0: (no value), adafruit:LED3MM
- added R1: 10k, rcl:0207/12
- renumbered U$2 to BBB
Connections:
- removed net N$1: LED1.K, RN2.1
- removed net VCC: IC1.16
- new net +3V3: IC1.16, R1.2
- new net /OE_RLY: IC1.13, R1.1
- new net DATA_RLY: BBB.11, IC1.14
- new net N$17: IC1.7, LED7.A
- net GND: now also RN2.1; no longer RN2.9
- net N$10: now also LED5.K, RN2.7; no longer IC1.1, LED2.A
- net N$11: now also LED2.A; no longer LED3.A
- net N$12: now also LED3.A; no longer LED4.A
- net N$13: now also LED4.A; no longer LED5.A
- net N$14: now also LED5.A; no longer LED6.A
- net N$15: now also LED7.K, RN2.9; no longer IC1.6, LED7.A
- net N$16: now also IC1.6, LED6.A; no longer IC1.7, LED8.A
- net N$2: now also LED1.K, RN2.3; no longer LED2.K, RN2.2
- net N$3: now also RN2.5; no longer RN2.3
- net N$4: now also LED2.K; no longer LED4.K
- net N$5: now also LED4.K, RN2.6; no longer LED5.K, RN2.5
- net N$6: now also RN2.8; no longer RN2.6
- net N$7: now also LED0.K, RN2.2; no longer LED7.K, RN2.7
- net N$8: now also IC1.15, LED0.A; no longer LED8.K, RN2.8
- net N$9: now also IC1.1; no longer IC1.15
Changed lines of the file:
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@@
 <attribute name="OC_NEWARK" value="unknown" x="-26.67" y="85.09" size="1.778" layer="27" display="off"/>
 </element>
-<element name="U$2" library="local" package="BEAGLEBONE_SHIELD" value="BEAGLEBONE_OUTLINE" x="-190.5" y="1.27"/>
+<element name="BBB" library="local" package="BEAGLEBONE_SHIELD" value="BEAGLEBONE_OUTLINE" x="-190.5" y="1.27"/>
 <element name="LED1" library="adafruit" package="LED3MM" value="" x="-187.96" y="-2.54"/>
 <element name="LED2" library="adafruit" package="LED3MM" value="" x="-187.96" y="-7.62"/>
@@
 <element name="LED7" library="adafruit" package="LED3MM" value="" x="-187.96" y="-33.02"/>
 <element name="LED8" library="adafruit" package="LED3MM" value="" x="-187.96" y="-38.1"/>
+<element name="LED0" library="adafruit" package="LED3MM" value="" x="-187.96" y="-43.18"/>
+<element name="R1" library="rcl" package="0207/12" value="10k" x="-182.88" y="-49.53"/>
 </elements>
 <signals>
 <signal name="GND">
+<contactref element="BBB" pad="90"/>
+<contactref element="BBB" pad="92"/>
+<contactref element="BBB" pad="48"/>
+<contactref element="RN2" pad="1"/>
 <contactref element="IC1" pad="8"/>
-<contactref element="U$2" pad="47"/>
-<contactref element="U$2" pad="48"/>
-<contactref element="U$2" pad="89"/>
-<contactref element="U$2" pad="90"/>
-<contactref element="U$2" pad="91"/>
-<contactref element="U$2" pad="92"/>
-<contactref element="U$2" pad="1"/>
-<contactref element="U$2" pad="2"/>
-<contactref element="RN2" pad="9"/>
+<contactref element="BBB" pad="2"/>
+<contactref element="BBB" pad="47"/>
+<contactref element="BBB" pad="89"/>
+<contactref element="BBB" pad="91"/>
+<contactref element="BBB" pad="1"/>
 <wire x1="-186.055" y1="20.32" x2="-188.595" y2="20.32" width="0" layer="19" extent="1-1"/>
 <wire x1="-140.335" y1="20.32" x2="-186.055" y2="20.32" width="0" layer="19" extent="1-1"/>
 <wire x1="-137.795" y1="20.32" x2="-140.335" y2="20.32" width="0" layer="19" extent="1-1"/>
 <wire x1="-140.335" y1="73.66" x2="-140.335" y2="20.32" width="0" layer="19" extent="1-1"/>
+<wire x1="-140.335" y1="76.2" x2="-140.335" y2="73.66" width="0" layer="19" extent="1-1"/>
 <wire x1="-137.795" y1="73.66" x2="-140.335" y2="73.66" width="0" layer="19" extent="1-1"/>
-<wire x1="-140.335" y1="76.2" x2="-140.335" y2="73.66" width="0" layer="19" extent="1-1"/>
-<wire x1="-137.795" y1="76.2" x2="-137.795" y2="73.66" width="0" layer="19" extent="1-1"/>
-<wire x1="-15.24" y1="92.71" x2="-137.795" y2="76.2" width="0" layer="19" extent="1-1"/>
-<wire x1="-15.24" y1="46.99" x2="-15.24" y2="92.71" width="0" layer="19" extent="1-1"/>
-</signal>
-<signal name="VCC">
-<contactref element="IC1" pad="16"/>
+<wire x1="-137.795" y1="76.2" x2="-140.335" y2="76.2" width="0" layer="19" extent="1-1"/>
+<wire x1="-35.56" y1="92.71" x2="-137.795" y2="76.2" width="0" layer="19" extent="1-1"/>
+<wire x1="-15.24" y1="46.99" x2="-35.56" y2="92.71" width="0" layer="19" extent="1-1"/>
 </signal>
 <signal name="VDD_3V3EXP">
-<contactref element="U$2" pad="49"/>
-<contactref element="U$2" pad="50"/>
+<contactref element="BBB" pad="49"/>
+<contactref element="BBB" pad="50"/>
 <wire x1="-137.795" y1="22.86" x2="-140.335" y2="22.86" width="0" layer="19" extent="1-1"/>
 </signal>
 <signal name="VDD_5V">
-<contactref element="U$2" pad="51"/>
-<contactref element="U$2" pad="52"/>
+<contactref element="BBB" pad="51"/>
+<contactref element="BBB" pad="52"/>
 <wire x1="-137.795" y1="25.4" x2="-140.335" y2="25.4" width="0" layer="19" extent="1-1"/>
 </signal>
 <signal name="SYS_5V">
-<contactref element="U$2" pad="53"/>
+<contactref element="BBB" pad="53"/>
 </signal>
 <signal name="AIN0">
-<contactref element="U$2" pad="85"/>
+<contactref element="BBB" pad="85"/>
 </signal>
-<signal name="N$1">
-<contactref element="LED1" pad="K"/>
-<contactref element="RN2" pad="1"/>
-<wire x1="-35.56" y1="92.71" x2="-186.69" y2="-2.54" width="0" layer="19" extent="1-1"/>
+<signal name="N$4">
+<contactref element="RN2" pad="4"/>
+<contactref element="LED2" pad="K"/>
+<wire x1="-27.94" y1="92.71" x2="-186.69" y2="-7.62" width="0" layer="19" extent="1-1"/>
 </signal>
 <signal name="N$2">
-<contactref element="LED2" pad="K"/>
-<contactref element="RN2" pad="2"/>
-<wire x1="-33.02" y1="92.71" x2="-186.69" y2="-7.62" width="0" layer="19" extent="1-1"/>
+<contactref element="RN2" pad="3"/>
+<contactref element="LED1" pad="K"/>
+<wire x1="-30.48" y1="92.71" x2="-186.69" y2="-2.54" width="0" layer="19" extent="1-1"/>
 </signal>
 <signal name="N$3">
+<contactref element="RN2" pad="5"/>
 <contactref element="LED3" pad="K"/>
-<contactref element="RN2" pad="3"/>
-<wire x1="-30.48" y1="92.71" x2="-186.69" y2="-12.7" width="0" layer="19" extent="1-1"/>
-</signal>
-<signal name="N$4">
-<contactref element="LED4" pad="K"/>
-<contactref element="RN2" pad="4"/>
-<wire x1="-27.94" y1="92.71" x2="-186.69" y2="-17.78" width="0" layer="19" extent="1-1"/>
+<wire x1="-25.4" y1="92.71" x2="-186.69" y2="-12.7" width="0" layer="19" extent="1-1"/>
 </signal>
 <signal name="N$5">
-<contactref element="LED5" pad="K"/>
-<contactref element="RN2" pad="5"/>
-<wire x1="-25.4" y1="92.71" x2="-186.69" y2="-22.86" width="0" layer="19" extent="1-1"/>
+<contactref element="RN2" pad="6"/>
+<contactref element="LED4" pad="K"/>
+<wire x1="-22.86" y1="92.71" x2="-186.69" y2="-17.78" width="0" layer="19" extent="1-1"/>
 </signal>
 <signal name="N$6">
+<contactref element="RN2" pad="8"/>
 <contactref element="LED6" pad="K"/>
-<contactref element="RN2" pad="6"/>
-<wire x1="-22.86" y1="92.71" x2="-186.69" y2="-27.94" width="0" layer="19" extent="1-1"/>
+<wire x1="-17.78" y1="92.71" x2="-186.69" y2="-27.94" width="0" layer="19" extent="1-1"/>
+</signal>
+<signal name="N$10">
+<contactref element="RN2" pad="7"/>
+<contactref element="LED5" pad="K"/>
+<wire x1="-20.32" y1="92.71" x2="-186.69" y2="-22.86" width="0" layer="19" extent="1-1"/>
+</signal>
+<signal name="+3V3">
+<contactref element="IC1" pad="16"/>
+<contactref element="R1" pad="2"/>
+<wire x1="-33.02" y1="54.61" x2="-176.53" y2="-49.53" width="0" layer="19" extent="1-1"/>
+</signal>
+<signal name="N$15">
+<contactref element="LED7" pad="K"/>
+<contactref element="RN2" pad="9"/>
+<wire x1="-15.24" y1="92.71" x2="-186.69" y2="-33.02" width="0" layer="19" extent="1-1"/>
 </signal>
 <signal name="N$7">
-<contactref element="LED7" pad="K"/>
-<contactref element="RN2" pad="7"/>
-<wire x1="-20.32" y1="92.71" x2="-186.69" y2="-33.02" width="0" layer="19" extent="1-1"/>
+<contactref element="RN2" pad="2"/>
+<contactref element="LED0" pad="K"/>
+<wire x1="-33.02" y1="92.71" x2="-186.69" y2="-43.18" width="0" layer="19" extent="1-1"/>
 </signal>
 <signal name="N$8">
-<contactref element="LED8" pad="K"/>
-<contactref element="RN2" pad="8"/>
-<wire x1="-17.78" y1="92.71" x2="-186.69" y2="-38.1" width="0" layer="19" extent="1-1"/>
+<contactref element="LED0" pad="A"/>
+<contactref element="IC1" pad="15"/>
+<wire x1="-30.48" y1="54.61" x2="-189.23" y2="-43.18" width="0" layer="19" extent="1-1"/>
 </signal>
 <signal name="N$9">
 <contactref element="LED1" pad="A"/>
-<contactref element="IC1" pad="15"/>
-<wire x1="-30.48" y1="54.61" x2="-189.23" y2="-2.54" width="0" layer="19" extent="1-1"/>
-</signal>
-<signal name="N$10">
-<contactref element="LED2" pad="A"/>
 <contactref element="IC1" pad="1"/>
-<wire x1="-33.02" y1="46.99" x2="-189.23" y2="-7.62" width="0" layer="19" extent="1-1"/>
+<wire x1="-33.02" y1="46.99" x2="-189.23" y2="-2.54" width="0" layer="19" extent="1-1"/>
 </signal>
 <signal name="N$11">
-<contactref element="LED3" pad="A"/>
+<contactref element="LED2" pad="A"/>
 <contactref element="IC1" pad="2"/>
-<wire x1="-30.48" y1="46.99" x2="-189.23" y2="-12.7" width="0" layer="19" extent="1-1"/>
+<wire x1="-30.48" y1="46.99" x2="-189.23" y2="-7.62" width="0" layer="19" extent="1-1"/>
 </signal>
 <signal name="N$12">
-<contactref element="LED4" pad="A"/>
+<contactref element="LED3" pad="A"/>
 <contactref element="IC1" pad="3"/>
-<wire x1="-27.94" y1="46.99" x2="-189.23" y2="-17.78" width="0" layer="19" extent="1-1"/>
+<wire x1="-27.94" y1="46.99" x2="-189.23" y2="-12.7" width="0" layer="19" extent="1-1"/>
 </signal>
 <signal name="N$13">
-<contactref element="LED5" pad="A"/>
+<contactref element="LED4" pad="A"/>
 <contactref element="IC1" pad="4"/>
-<wire x1="-25.4" y1="46.99" x2="-189.23" y2="-22.86" width="0" layer="19" extent="1-1"/>
+<wire x1="-25.4" y1="46.99" x2="-189.23" y2="-17.78" width="0" layer="19" extent="1-1"/>
 </signal>
 <signal name="N$14">
-<contactref element="LED6" pad="A"/>
+<contactref element="LED5" pad="A"/>
 <contactref element="IC1" pad="5"/>
-<wire x1="-22.86" y1="46.99" x2="-189.23" y2="-27.94" width="0" layer="19" extent="1-1"/>
-</signal>
-<signal name="N$15">
-<contactref element="LED7" pad="A"/>
-<contactref element="IC1" pad="6"/>
-<wire x1="-20.32" y1="46.99" x2="-189.23" y2="-33.02" width="0" layer="19" extent="1-1"/>
+<wire x1="-22.86" y1="46.99" x2="-189.23" y2="-22.86" width="0" layer="19" extent="1-1"/>
 </signal>
 <signal name="N$16">
-<contactref element="LED8" pad="A"/>
+<contactref element="LED6" pad="A"/>
+<contactref element="IC1" pad="6"/>
+<wire x1="-20.32" y1="46.99" x2="-189.23" y2="-27.94" width="0" layer="19" extent="1-1"/>
+</signal>
+<signal name="N$17">
+<contactref element="LED7" pad="A"/>
 <contactref element="IC1" pad="7"/>
-<wire x1="-17.78" y1="46.99" x2="-189.23" y2="-38.1" width="0" layer="19" extent="1-1"/>
+<wire x1="-17.78" y1="46.99" x2="-189.23" y2="-33.02" width="0" layer="19" extent="1-1"/>
+</signal>
+<signal name="DATA_RLY">
+<contactref element="IC1" pad="14"/>
+<contactref element="BBB" pad="11"/>
+<wire x1="-27.94" y1="54.61" x2="-186.055" y2="33.02" width="0" layer="19" extent="1-1"/>
+</signal>
+<signal name="/OE_RLY">
+<contactref element="IC1" pad="13"/>
+<contactref element="R1" pad="1"/>
+<wire x1="-25.4" y1="54.61" x2="-189.23" y2="-49.53" width="0" layer="19" extent="1-1"/>
 </signal>
 </signals>

Commit message: again
Parts:
- moved RN2 108.4 mm to (81.3, 73.7)
Changed lines of the file:
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@@
 <?xml version="1.0" encoding="utf-8"?>
 <!DOCTYPE eagle SYSTEM "eagle.dtd">
-<eagle version="7.5.2">
+<eagle version="6.5.0">
 <drawing>
 <settings>
@@
 <pass name="Default">
 <param name="RoutingGrid" value="50mil"/>
-<param name="AutoGrid" value="1"/>
-<param name="Efforts" value="0"/>
-<param name="TopRouterVariant" value="1"/>
 <param name="tpViaShape" value="round"/>
-<param name="PrefDir.1" value="a"/>
+<param name="PrefDir.1" value="|"/>
 <param name="PrefDir.2" value="0"/>
 <param name="PrefDir.3" value="0"/>
@@
 <param name="PrefDir.14" value="0"/>
 <param name="PrefDir.15" value="0"/>
-<param name="PrefDir.16" value="a"/>
+<param name="PrefDir.16" value="-"/>
 <param name="cfVia" value="8"/>
 <param name="cfNonPref" value="5"/>
@@
 <attribute name="OC_NEWARK" value="unknown" x="-66.04" y="81.28" size="1.778" layer="27" display="off"/>
 </element>
-<element name="RN2" library="resistor-sil" package="SIL9" value="" x="-25.4" y="92.71">
-<attribute name="MF" value="" x="-25.4" y="92.71" size="1.778" layer="27" display="off"/>
-<attribute name="OC_FARNELL" value="unknown" x="-25.4" y="92.71" size="1.778" layer="27" display="off"/>
-<attribute name="MPN" value="" x="-25.4" y="92.71" size="1.778" layer="27" display="off"/>
-<attribute name="OC_NEWARK" value="unknown" x="-25.4" y="92.71" size="1.778" layer="27" display="off"/>
+<element name="RN2" library="resistor-sil" package="SIL9" value="" x="81.28" y="73.66">
+<attribute name="MF" value="" x="81.28" y="73.66" size="1.778" layer="27" display="off"/>
+<attribute name="OC_FARNELL" value="unknown" x="81.28" y="73.66" size="1.778" layer="27" display="off"/>
+<attribute name="MPN" value="" x="81.28" y="73.66" size="1.778" layer="27" display="off"/>
+<attribute name="OC_NEWARK" value="unknown" x="81.28" y="73.66" size="1.778" layer="27" display="off"/>
 </element>
 <element name="SV1" library="con-lstb" package="MA05-2" value="" x="-46.99" y="85.09">
@@
 <wire x1="-137.795" y1="73.66" x2="-140.335" y2="73.66" width="0" layer="19" extent="1-1"/>
 <wire x1="-137.795" y1="76.2" x2="-140.335" y2="76.2" width="0" layer="19" extent="1-1"/>
-<wire x1="-35.56" y1="92.71" x2="-137.795" y2="76.2" width="0" layer="19" extent="1-1"/>
-<wire x1="-15.24" y1="46.99" x2="-35.56" y2="92.71" width="0" layer="19" extent="1-1"/>
+<wire x1="71.12" y1="73.66" x2="-137.795" y2="76.2" width="0" layer="19" extent="1-1"/>
+<wire x1="-15.24" y1="46.99" x2="71.12" y2="73.66" width="0" layer="19" extent="1-1"/>
 </signal>
 <signal name="VDD_3V3EXP">
@@
 <contactref element="RN2" pad="4"/>
 <contactref element="LED2" pad="K"/>
-<wire x1="-27.94" y1="92.71" x2="-186.69" y2="-7.62" width="0" layer="19" extent="1-1"/>
+<wire x1="78.74" y1="73.66" x2="-186.69" y2="-7.62" width="0" layer="19" extent="1-1"/>
 </signal>
 <signal name="N$2">
 <contactref element="RN2" pad="3"/>
 <contactref element="LED1" pad="K"/>
-<wire x1="-30.48" y1="92.71" x2="-186.69" y2="-2.54" width="0" layer="19" extent="1-1"/>
+<wire x1="76.2" y1="73.66" x2="-186.69" y2="-2.54" width="0" layer="19" extent="1-1"/>
 </signal>
 <signal name="N$3">
 <contactref element="RN2" pad="5"/>
 <contactref element="LED3" pad="K"/>
-<wire x1="-25.4" y1="92.71" x2="-186.69" y2="-12.7" width="0" layer="19" extent="1-1"/>
+<wire x1="81.28" y1="73.66" x2="-186.69" y2="-12.7" width="0" layer="19" extent="1-1"/>
 </signal>
 <signal name="N$5">
 <contactref element="RN2" pad="6"/>
 <contactref element="LED4" pad="K"/>
-<wire x1="-22.86" y1="92.71" x2="-186.69" y2="-17.78" width="0" layer="19" extent="1-1"/>
+<wire x1="83.82" y1="73.66" x2="-186.69" y2="-17.78" width="0" layer="19" extent="1-1"/>
 </signal>
 <signal name="N$6">
 <contactref element="RN2" pad="8"/>
 <contactref element="LED6" pad="K"/>
-<wire x1="-17.78" y1="92.71" x2="-186.69" y2="-27.94" width="0" layer="19" extent="1-1"/>
+<wire x1="88.9" y1="73.66" x2="-186.69" y2="-27.94" width="0" layer="19" extent="1-1"/>
 </signal>
 <signal name="N$10">
 <contactref element="RN2" pad="7"/>
 <contactref element="LED5" pad="K"/>
-<wire x1="-20.32" y1="92.71" x2="-186.69" y2="-22.86" width="0" layer="19" extent="1-1"/>
+<wire x1="86.36" y1="73.66" x2="-186.69" y2="-22.86" width="0" layer="19" extent="1-1"/>
 </signal>
 <signal name="+3V3">
@@
 <contactref element="RN2" pad="2"/>
 <contactref element="LED0" pad="K"/>
-<wire x1="-33.02" y1="92.71" x2="-186.69" y2="-43.18" width="0" layer="19" extent="1-1"/>
+<wire x1="73.66" y1="73.66" x2="-186.69" y2="-43.18" width="0" layer="19" extent="1-1"/>
 </signal>
 <signal name="N$8">
@@
 <contactref element="LED7" pad="K"/>
 <contactref element="RN2" pad="9"/>
-<wire x1="-15.24" y1="92.71" x2="-186.69" y2="-33.02" width="0" layer="19" extent="1-1"/>
+<wire x1="91.44" y1="73.66" x2="-186.69" y2="-33.02" width="0" layer="19" extent="1-1"/>
 </signal>
 </signals>
